Commit message: 增加新任务点，解决印章穿模

File: models/urdf/装配体1.SLDASM/scene2_solidworks_import.urdf (robot description, URDF)
Before this commit: robot scene2_solidworks_stamp_arm, 6 links, 5 joints
Links:
- link base_link: mass 48.035 -> 48.0345575191895
- link link_2: mass 1.4576 -> 1.45761059759436
- link link_3: mass 1.4576 -> 1.45761059759436
- link link_4: mass 0.57754 -> 0.577535390627309
- link link_5: mass 0.30316 -> 0.303163691071415
Joints:
- joint joint_2: limit lower=-3.14159265358979 upper=3.14159265358979 effort=15 velocity=2 -> lower=-3.14159265358979 upper=3.14159265358979 effort=20 velocity=2
- joint joint_3: limit lower=-3.14159265358979 upper=3.14159265358979 effort=15 velocity=2 -> lower=-3.14159265358979 upper=3.14159265358979 effort=20 velocity=2
- joint joint_4: limit lower=-3.14159265358979 upper=3.14159265358979 effort=15 velocity=2 -> lower=-3.14159265358979 upper=3.14159265358979 effort=20 velocity=2
- joint joint_5: origin xyz=0.11 0 0 rpy=1.5708 0 0 -> xyz=0.11 -0.01 0.0 rpy=1.5708 0 0

File: models/urdf/装配体1.SLDASM/scene2_solidworks_pd_tracking.urdf (robot description, URDF)
Before this commit: robot 装配体1.SLDASM, 6 links, 5 joints
Links:
- link base_link: geometry collision mesh filename=meshes/base_link.STL; visual mesh filename=meshes/base_link.STL
- link link_1: geometry collision mesh filename=meshes/link_1.STL; visual mesh filename=meshes/link_1.STL
- link link_2: geometry collision mesh filename=meshes/link_2.STL; visual mesh filename=meshes/link_2.STL
- link link_3: geometry collision mesh filename=meshes/link_3.STL; visual mesh filename=meshes/link_3.STL
- link link_4: geometry collision mesh filename=meshes/link_4.STL; visual mesh filename=meshes/link_4.STL
- link link_5: geometry collision mesh filename=meshes/link_5.STL; visual mesh filename=meshes/link_5.STL
Joints:
- joint joint_2: limit lower=0 upper=1.5708 effort=20 velocity=2 -> lower=-3.14159265358979 upper=3.14159265358979 effort=20 velocity=2
- joint joint_3: limit lower=-1.5708 upper=1.5708 effort=20 velocity=2 -> lower=-3.14159265358979 upper=3.14159265358979 effort=20 velocity=2
- joint joint_4: limit lower=-1.5708 upper=1.5708 effort=20 velocity=2 -> lower=-3.14159265358979 upper=3.14159265358979 effort=20 velocity=2
- joint joint_5: origin xyz=0.11 -0.02 0 rpy=1.5708 0 0 -> xyz=0.11 -0.01 0.0 rpy=1.5708 0 0
